Commit message: Cleaned up repo.

File: digit.urdf (robot description, URDF)
Before this commit: robot digit, 41 links, 35 joints
Links:
- removed link left-achilles-rod_link
- removed link left-toe-A-rod_link
- removed link left-toe-B-rod_link
- removed link right-achilles-rod_link
- removed link right-toe-A-rod_link
- removed link right-toe-B-rod_link
- link left-elbow_link: geometry collision cylinder length=0.1565 radius=0.013; collision sphere radius=0.015
- link left-foot_link: geometry collision sphere radius=1e-7; collision sphere radius=1e-7
- link left-shoulder-pitch_link: geometry collision cylinder length=0.07 radius=0.038; visual mesh filename=obj/arm-l2.obj
- link left-shoulder-roll_link: geometry visual mesh filename=obj/arm-l1.obj
- link left-shoulder-yaw_link: geometry collision cylinder length=0.04 radius=0.03; collision cylinder length=0.0675 radius=0.038
- link right-elbow_link: geometry collision cylinder length=0.1565 radius=0.013; collision sphere radius=0.015
- link right-foot_link: geometry collision sphere radius=1e-7; collision sphere radius=1e-7
- link right-shoulder-pitch_link: geometry collision cylinder length=0.07 radius=0.038; visual mesh filename=obj/arm-l2-xz.obj
- link right-shoulder-roll_link: geometry visual mesh filename=obj/arm-l1-xz.obj
- link right-shoulder-yaw_link: geometry collision cylinder length=0.04 radius=0.03; collision cylinder length=0.0675 radius=0.038
Joints:
- joint base_joint: origin xyz=0 0 0 rpy=-0 0 -0 -> xyz=0 0 0 rpy=0 0 0
- joint left-elbow_joint: origin xyz=0 -0.0385 0.185 rpy=1.5708 0 0 -> xyz=0 -0.0385 0.185 rpy=1.5707963267948966 -0.3926990816987242 6.0084837121965e-17
- joint left-foot_joint: origin xyz=0 -0.05456 -0.0315 rpy=-1.0472 0 -1.5708 -> xyz=0 -0.05456 -0.0315 rpy=-4.440892098500625e-16 -1.0471975511965976 -1.5707963267948961
- joint left-hand_joint: origin xyz=0.369 0 -0.07912 rpy=1.5708 0 -0.174533 -> xyz=0.369 0 -0.07912 rpy=1.5707963267948963 0.17453292519943295 -4.2275625162475e-17
- joint left-heel-spring_joint: origin xyz=-0.01766 -0.029456 0.00104 rpy=0.07801622 0.005585054 2.719223 -> xyz=-0.01766 -0.029456 0.00104 rpy=-0.06890726319112118 -0.03703539652316154 2.720717602917085
- joint left-hip-pitch_joint: origin xyz=0 0.004 0.068 rpy=1.5708 0 0 -> xyz=0 0.004 0.068 rpy=-1.5707963267948966 -0.7853981633974483 3.141592653589793
- joint left-hip-roll_joint: origin xyz=-0.001 0.091 0 rpy=0 -1.5708 0 -> xyz=-0.001 0.091 0 rpy=1.570796326794897 -1.1955505376161157 -1.570796326794897
- joint left-hip-yaw_joint: origin xyz=-0.0505 0 0.044 rpy=0 -1.5708 0 -> xyz=-0.0505 0 0.044 rpy=0.0 -1.5707963267948966 0.0
- joint left-knee_joint: origin xyz=-0.085 0.085 0.0045 rpy=0 0 0.785398 -> xyz=0.12 0 0.0045 rpy=0.0 0.0 -1.5707963267948966
- joint left-shin_joint: type continuous -> fixed
- joint left-shoulder-pitch_joint: origin xyz=-0.00317 -0.011055 0.0555 rpy=1.5708 0 -0.279253 -> xyz=-0.00317 -0.011055 0.0555 rpy=1.5707963267948966 0.7853981633974485 -0.2792526803190933
- joint left-shoulder-roll_joint: origin xyz=-0.001 0.12 0.4 rpy=-0.174533 -1.5708 0 -> xyz=-0.001 0.12 0.4 rpy=-1.5707963267948954 -1.3962634015954636 1.5707963267948954
- joint left-shoulder-yaw_joint: origin xyz=0 -0.165 -0.1 rpy=1.5708 0 0 -> xyz=0 -0.165 -0.1 rpy=1.5707963267948966 -0.0 0.0
- joint left-tarsus_joint: origin xyz=0.434759 0.02 0 rpy=0 0 1.79769 -> xyz=0.434759 0.02 0 rpy=0.0 -0.0 1.7976891295541595
- joint left-toe-A_joint: origin xyz=0.059 -0.034 -0.0276 rpy=-3.14159 0 1.5526449 -> xyz=0.059 -0.034 -0.0276 rpy=-3.141592653589793 1.2244450599234578e-16 -1.5526449025741558
- joint left-toe-B_joint: origin xyz=0.111 -0.034 0.0276 rpy=0 0 -1.5526449 -> xyz=0.111 -0.034 0.0276 rpy=0.0 0.0 -1.5526449025741558
- joint left-toe-pitch_joint: origin xyz=0.408 -0.04 0 rpy=0 0 1.2522737 -> xyz=0.408 -0.04 0 rpy=0.0 -0.0 1.2522737383059317
- joint left-toe-roll_joint: origin xyz=0 0 0 rpy=0 1.5708 0 -> xyz=0 0 0 rpy=-0.0 1.5707963267948966 0.0
- joint right-elbow_joint: origin xyz=0 0.0385 0.185 rpy=-1.5708 0 0 -> xyz=0 0.0385 0.185 rpy=-1.5707963267948966 -0.3926990816987242 -6.0084837121965e-17
- joint right-foot_joint: origin xyz=0 0.05456 -0.0315 rpy=1.0472 0 1.5708 -> xyz=0 0.05456 -0.0315 rpy=4.440892098500625e-16 -1.0471975511965976 1.5707963267948961
- joint right-hand_joint: origin xyz=0.369 0 -0.07912 rpy=-1.5708 0 0.174533 -> xyz=0.369 0 -0.07912 rpy=-1.5707963267948963 0.17453292519943295 4.2275625162475e-17
- joint right-heel-spring_joint: origin xyz=-0.01766 0.029456 0.00104 rpy=-0.07801622 0.005585054 -2.719223 -> xyz=-0.01766 0.029456 0.00104 rpy=0.06890726319112118 -0.03703539652316154 -2.720717602917085
- joint right-hip-pitch_joint: origin xyz=0 -0.004 0.068 rpy=-1.5708 0 0 -> xyz=0 -0.004 0.068 rpy=1.5707963267948966 -0.7853981633974483 -3.141592653589793
- joint right-hip-roll_joint: origin xyz=-0.001 -0.091 0 rpy=0 -1.5708 0 -> xyz=-0.001 -0.091 0 rpy=-1.570796326794897 -1.1955505376161157 1.570796326794897
- joint right-hip-yaw_joint: origin xyz=-0.0505 0 0.044 rpy=0 -1.5708 0 -> xyz=-0.0505 0 0.044 rpy=0.0 -1.5707963267948966 0.0
- joint right-knee_joint: origin xyz=-0.085 -0.085 0.0045 rpy=0 0 -0.785398 -> xyz=0.12 0 0.0045 rpy=0.0 -0.0 1.5707963267948966
- joint right-shin_joint: type continuous -> fixed
- joint right-shoulder-pitch_joint: origin xyz=-0.00317 0.011055 0.0555 rpy=-1.5708 0 0.279253 -> xyz=-0.00317 0.011055 0.0555 rpy=-1.5707963267948966 0.7853981633974485 0.2792526803190933
- joint right-shoulder-roll_joint: origin xyz=-0.001 -0.12 0.4 rpy=0.174533 -1.5708 0 -> xyz=-0.001 -0.12 0.4 rpy=1.5707963267948954 -1.3962634015954636 -1.5707963267948954
- joint right-shoulder-yaw_joint: origin xyz=0 0.165 -0.1 rpy=-1.5708 0 0 -> xyz=0 0.165 -0.1 rpy=-1.5707963267948966 0.0 0.0
- joint right-tarsus_joint: origin xyz=0.434759 -0.02 0 rpy=0 0 -1.79769 -> xyz=0.434759 -0.02 0 rpy=0.0 0.0 -1.7976891295541595
- joint right-toe-A_joint: origin xyz=0.059 0.034 -0.0276 rpy=3.14159 0 -1.5526449 -> xyz=0.059 0.034 -0.0276 rpy=3.141592653589793 1.2244450599234578e-16 1.5526449025741558
- joint right-toe-B_joint: origin xyz=0.111 0.034 0.0276 rpy=0 0 1.5526449 -> xyz=0.111 0.034 0.0276 rpy=0.0 -0.0 1.5526449025741558
- joint right-toe-pitch_joint: origin xyz=0.408 0.04 0 rpy=0 0 -1.2522737 -> xyz=0.408 0.04 0 rpy=0.0 0.0 -1.2522737383059317
- joint right-toe-roll_joint: origin xyz=0 0 0 rpy=0 1.5708 0 -> xyz=0 0 0 rpy=-0.0 1.5707963267948966 0.0
